File: keyboardpcb.kicad_pcb (KiCad board)
At the start: 2 copper layers, 155 parts, among them J1 AVR-ISP-6, K1 ESC, K10 #9, K11 #0, K12 -_, K13 =+, K14 BSPC, K15 PGUP, K16 TAB, K17 Q, K18 W, K19 E, K2 #1, K20 R, K21 T, K22 Y, K23 U, K24 I, K25 O, K26 P, K27 [{, K28 ]}, K29 \|, K3 #2, K30 PGDN, K31 CAPS, K32 A, K33 S, K34 D, K35 F, K36 G, K37 H, K38 J, K39 K, K4 #3, K40 L, K41 ;:, K42 '", K43 ENT, K44 INS, K45 LSHFT, K46 Z, K47 X, K48 C, K49 V, K5 #4, K50 B, K51 N, K52 M, K53 ,<, K54 .>, K55 /?, K56 RSHFT, K57 UP, K58 DEL, K59 CTRL, K6 #5, K60 WIN, K61 LALT, K62 SPC, K63 RALT, K64 FN, K65 LEFT, K66 DOWN, K67 RGHT, K7 #6, K8 #7, K9 #8, SW1 SW_Push_Reset, U1 ATmega32U4-A, U2 PRTR5V0U2X, X1 XTAL

Commit message: Final Complete
Parts:
- added FB1: 60@100MHz, Inductor_SMD:L_0805_2012Metric_Pad1.15x1.40mm_HandSolder, B.Cu at (159.9, 2.00)
- added G***: LOGO, LOGO, F.Cu at (46.5, 49.4)
- added G***: LOGO, LOGO, F.Cu at (103.9, 83.1)
- added G***: LOGO, LOGO, B.Cu at (112.9, 91.4)
- added G***: LOGO, LOGO, B.Cu at (122.9, 85.7)
- added G***: LOGO, LOGO, B.Cu at (105.6, 89.9)
- added G***: LOGO, LOGO, B.Cu at (111.9, 83.7)
- K1, K12, K13, K15, K17, K18, K19, K20, K21, K22, K23, K24, K25, K26, K27, K28, K30, K32, K33, K34, K35, K36, K37, K38, K39, K40, K44, K46, K47, K48, K49, K50, K51, K52, K53, K54, K55, K57, K58, K64, K65, K66, K67: footprint MX_Alps_Hybrid:MX-1U -> MX_Alps_Hybrid:MX-1U-NoLED
- K10: value #9 -> 9; footprint MX_Alps_Hybrid:MX-1U -> MX_Alps_Hybrid:MX-1U-NoLED
- K11: value #0 -> 0; footprint MX_Alps_Hybrid:MX-1U -> MX_Alps_Hybrid:MX-1U-NoLED
- K14: footprint MX_Alps_Hybrid:MX-2U -> MX_Alps_Hybrid:MX-2U-NoLED
- K16, K29, K59, K61: footprint MX_Alps_Hybrid:MX-1.5U -> MX_Alps_Hybrid:MX-1.5U-NoLED
- K2: value #1 -> 1; footprint MX_Alps_Hybrid:MX-1U -> MX_Alps_Hybrid:MX-1U-NoLED
- K3: value #2 -> 2; footprint MX_Alps_Hybrid:MX-1U -> MX_Alps_Hybrid:MX-1U-NoLED
- K31, K56: footprint MX_Alps_Hybrid:MX-1.75U -> MX_Alps_Hybrid:MX-1.75U-NoLED
- K4: value #3 -> 3; footprint MX_Alps_Hybrid:MX-1U -> MX_Alps_Hybrid:MX-1U-NoLED
- K41: value ;: -> ; :; footprint MX_Alps_Hybrid:MX-1U -> MX_Alps_Hybrid:MX-1U-NoLED
- K42: value '" -> ' "; footprint MX_Alps_Hybrid:MX-1U -> MX_Alps_Hybrid:MX-1U-NoLED
- K43, K45: footprint MX_Alps_Hybrid:MX-2.25U -> MX_Alps_Hybrid:MX-2.25U-NoLED
- K5: value #4 -> 4; footprint MX_Alps_Hybrid:MX-1U -> MX_Alps_Hybrid:MX-1U-NoLED
- K6: value #5 -> 5; footprint MX_Alps_Hybrid:MX-1U -> MX_Alps_Hybrid:MX-1U-NoLED
- K60, K63: footprint MX_Alps_Hybrid:MX-1.25U -> MX_Alps_Hybrid:MX-1.25U-NoLED
- K62: footprint MX_Alps_Hybrid:MX-6.5U -> MX_Alps_Hybrid:MX-6.5U-NoLED
- K7: value #6 -> 6; footprint MX_Alps_Hybrid:MX-1U -> MX_Alps_Hybrid:MX-1U-NoLED
- K8: value #7 -> 7; footprint MX_Alps_Hybrid:MX-1U -> MX_Alps_Hybrid:MX-1U-NoLED
- K9: value #8 -> 8; footprint MX_Alps_Hybrid:MX-1U -> MX_Alps_Hybrid:MX-1U-NoLED
- moved SW1 125.6 mm to (192.9, 85.6), turned to 0 degrees
- moved J1 122.0 mm to (203.7, 80.7)
- moved R2 110.5 mm to (186.4, 87.5), turned to 0 degrees
- moved C2 104.2 mm to (181.7, 87.5)
- moved D52 101.7 mm to (152.1, 72.8)
- moved X1 101.6 mm to (177.1, 86.2), turned to 90 degrees
- moved D23 101.5 mm to (138.6, 34.6)
- moved D38 101.5 mm to (143.4, 53.7)
- moved D11 100.6 mm to (192.6, 15.7)
- moved D14 100.6 mm to (259.2, 15.7)
- moved D15 100.6 mm to (287.8, 15.7)
- moved D20 100.6 mm to (87.8, 34.8)
- moved D21 100.6 mm to (106.8, 34.8)
- moved D28 100.6 mm to (240.2, 34.8)
- moved D29 100.6 mm to (264.0, 34.8)
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Connections:
- net Net-(U2-IO1) renamed DP
- net Net-(U2-IO2) renamed DN
- C2 pad 2: Net-(C2-Pad2) -> GND
- C3 pad 2: Net-(C2-Pad2) -> GND
- U1 pad 1: row0 -> row3
- U1 pad 36: col6 -> row4
- U1 pad 38: row1 -> col6
- U1 pad 39: row4 -> row0
- U1 pad 40: row3 -> row1
- USB1 pad 13: GND -> Earth
- X1 pad 2: Net-(C2-Pad2) -> GND
- X1 pad 4: Net-(C2-Pad2) -> GND
Routing:
- net row0: track 0.00 -> 506.5 mm, vias 0 -> 2
- net row1: track 0.00 -> 476.4 mm, vias 0 -> 2
- net row2: track 0.00 -> 455.9 mm, vias 0 -> 2
- net row4: track 0.00 -> 300.7 mm, vias 0 -> 2
- net row3: track 0.00 -> 288.1 mm, vias 0 -> 2
- net GND: track 0.00 -> 271.1 mm, vias 0 -> 69
- net col0: track 0.00 -> 250.5 mm, vias 0 -> 1
- net col1: track 0.00 -> 229.8 mm, vias 0 -> 1
- net col14: track 0.00 -> 223.5 mm, vias 0 -> 1
- net col13: track 0.00 -> 213.3 mm, vias 0 -> 1
- net col2: track 0.00 -> 198.5 mm, vias 0 -> 1
- net +5V: track 0.00 -> 195.6 mm, vias 0 -> 9
- net col12: track 0.00 -> 193.4 mm, vias 0 -> 1
- net col11: track 0.00 -> 168.0 mm, vias 0 -> 1
- net col3: track 0.00 -> 166.1 mm, vias 0 -> 1
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- added copper zone on B.Cu, net Earth
- added copper zone on F.Cu, net Earth
- added copper zone on B.Cu, net GND
- added copper zone on F.Cu, net GND
Other:
- board outline added: 304.8 x 102 mm

Commit message: PCB Footprint switched to MX only, layout changed
Parts:
- K1, K10, K11, K12, K13, K15, K17, K18, K19, K2, K20, K21, K22, K23, K24, K25, K26, K27, K28, K3, K30, K32, K33, K34, K35, K36, K37, K38, K39, K4, K40, K41, K42, K44, K46, K47, K48, K49, K5, K50, K51, K52, K53, K54, K55, K57, K58, K6, K65, K66, K67, K7, K8, K9: footprint MX_Alps_Hybrid:MX-1U-NoLED -> Mx_Only:MX-Solderable-1U
- K14: footprint MX_Alps_Hybrid:MX-2U-NoLED -> Mx_Only:MX-Solderable-2U
- K16, K29, K59, K61: footprint MX_Alps_Hybrid:MX-1.5U-NoLED -> Mx_Only:MX-Solderable-1.5U
- K31, K56: footprint MX_Alps_Hybrid:MX-1.75U-NoLED -> Mx_Only:MX-Solderable-1.75U
- K43, K45: footprint MX_Alps_Hybrid:MX-2.25U-NoLED -> Mx_Only:MX-Solderable-2.25U
- K60, K63: footprint MX_Alps_Hybrid:MX-1.25U-NoLED -> Mx_Only:MX-Solderable-1.25U
- K62: footprint MX_Alps_Hybrid:MX-6.5U-NoLED -> Mx_Only:MX-Solderable-6.25U
- K64: footprint MX_Alps_Hybrid:MX-1U-NoLED -> Mx_Only:MX-Solderable-1.25U
- moved K63 4.46 mm to (211.1, 86.5)
- moved D63 4.46 mm to (204.8, 92.0)
- moved D64 2.13 mm to (228.6, 92.4)
- moved J1 2.09 mm to (201.9, 79.6)
- moved K62 2.09 mm to (139.7, 86.5)
- moved K64 2.09 mm to (234.9, 86.5)
- moved D62 2.08 mm to (133.3, 92.1)
- moved D57 0.38 mm to (269.1, 73.1)
- moved D58 0.38 mm to (288.1, 73.1)
- moved D43 0.38 mm to (257.2, 54.0)
- moved D44 0.38 mm to (288.1, 54.0)
- moved D15 0.38 mm to (288.1, 15.9)
- moved D29 0.38 mm to (264.3, 35.0)
- moved D30 0.38 mm to (288.1, 35.0)
- moved D66 0.38 mm to (269.1, 92.1)
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Routing:
- net col6: track 103.0 -> 106.5 mm
- net col10: track 151.4 -> 148.2 mm
- net GND: track 271.1 -> 274.3 mm, vias 69 -> 65
- net col11: track 168.0 -> 165.1 mm
- net MOSI: track 42.3 -> 39.7 mm
- net MISO: track 38.8 -> 36.1 mm
- net SCK: track 40.0 -> 37.3 mm
- net col12: track 193.4 -> 195.1 mm
- net col3: track 166.1 -> 167.7 mm
- net col8: track 115.2 -> 116.6 mm
- net col9: track 136.2 -> 135.0 mm
- net col13: track 213.3 -> 214.5 mm
- net VCC: track 24.2 -> 23.1 mm
- net col14: track 223.5 -> 224.3 mm
- net Net-(USB1-CC2): track 4.48 -> 5.16 mm
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