File: matrix.kicad_sch (KiCad schematic)
At the start: 134 parts, among them K1 ESC, K10 #9, K11 #0, K12 -_, K13 =+, K14 BSPC, K15 PGUP, K16 TAB, K17 Q, K18 W, K19 E, K2 #1, K20 R, K21 T, K22 Y, K23 U, K24 I, K25 O, K26 P, K27 [{, K28 ]}, K29 \|, K3 #2, K30 PGDN, K31 CAPS, K32 A, K33 S, K34 D, K35 F, K36 G, K37 H, K38 J, K39 K, K4 #3, K40 L, K41 ;:, K42 '", K43 ENT, K44 INS, K45 LSHFT, K46 Z, K47 X, K48 C, K49 V, K5 #4, K50 B, K51 N, K52 M, K53 ,<, K54 .>, K55 /?, K56 RSHFT, K57 UP, K58 DEL, K59 CTRL, K6 #5, K60 WIN, K61 LALT, K62 SPC, K63 RALT, K64 FN, K65 LEFT, K66 DOWN, K67 RGHT, K7 #6, K8 #7, K9 #8

Commit message: Matrix and pcb layout
Parts:
- D1, D10, D11, D12, D13, D14, D15, D16, D17, D18, D19, D2, D20, D21, D22, D23, D24, D25, D26, D27, D28, D29, D3, D30, D31, D32, D33, D34, D35, D36, D37, D38, D39, D4, D40, D41, D42, D43, D44, D45, D46, D47, D48, D49, D5, D50, D51, D52, D53, D54, D55, D56, D57, D58, D59, D6, D60, D61, D62, D63, D64, D65, D66, D67, D7, D8, D9: footprint (none) -> Diode_SMD:D_SOD-123
- K1, K10, K11, K12, K13, K15, K17, K18, K19, K2, K20, K21, K22, K23, K24, K25, K26, K27, K28, K3, K30, K32, K33, K34, K35, K36, K37, K38, K39, K4, K40, K41, K42, K44, K46, K47, K48, K49, K5, K50, K51, K52, K53, K54, K55, K57, K58, K6, K64, K65, K66, K67, K7, K8, K9: footprint (none) -> MX_Alps_Hybrid:MX-1U
- K14: footprint (none) -> MX_Alps_Hybrid:MX-2U
- K16, K29, K59, K61: footprint (none) -> MX_Alps_Hybrid:MX-1.5U
- K31, K56: footprint (none) -> MX_Alps_Hybrid:MX-1.75U
- K43, K45: footprint (none) -> MX_Alps_Hybrid:MX-2.25U
- K60, K63: footprint (none) -> MX_Alps_Hybrid:MX-1.25U
- K62: footprint (none) -> MX_Alps_Hybrid:MX-6.5U

Commit message: Final Complete
Parts:
- K1, K12, K13, K15, K17, K18, K19, K20, K21, K22, K23, K24, K25, K26, K27, K28, K30, K32, K33, K34, K35, K36, K37, K38, K39, K40, K44, K46, K47, K48, K49, K50, K51, K52, K53, K54, K55, K57, K58, K64, K65, K66, K67: footprint MX_Alps_Hybrid:MX-1U -> MX_Alps_Hybrid:MX-1U-NoLED
- K10: value #9 -> 9; footprint MX_Alps_Hybrid:MX-1U -> MX_Alps_Hybrid:MX-1U-NoLED
- K11: value #0 -> 0; footprint MX_Alps_Hybrid:MX-1U -> MX_Alps_Hybrid:MX-1U-NoLED
- K14: footprint MX_Alps_Hybrid:MX-2U -> MX_Alps_Hybrid:MX-2U-NoLED
- K16, K29, K59, K61: footprint MX_Alps_Hybrid:MX-1.5U -> MX_Alps_Hybrid:MX-1.5U-NoLED
- K2: value #1 -> 1; footprint MX_Alps_Hybrid:MX-1U -> MX_Alps_Hybrid:MX-1U-NoLED
- K3: value #2 -> 2; footprint MX_Alps_Hybrid:MX-1U -> MX_Alps_Hybrid:MX-1U-NoLED
- K31, K56: footprint MX_Alps_Hybrid:MX-1.75U -> MX_Alps_Hybrid:MX-1.75U-NoLED
- K4: value #3 -> 3; footprint MX_Alps_Hybrid:MX-1U -> MX_Alps_Hybrid:MX-1U-NoLED
- K41: value ;: -> ; :; footprint MX_Alps_Hybrid:MX-1U -> MX_Alps_Hybrid:MX-1U-NoLED
- K42: value '" -> ' "; footprint MX_Alps_Hybrid:MX-1U -> MX_Alps_Hybrid:MX-1U-NoLED
- K43, K45: footprint MX_Alps_Hybrid:MX-2.25U -> MX_Alps_Hybrid:MX-2.25U-NoLED
- K5: value #4 -> 4; footprint MX_Alps_Hybrid:MX-1U -> MX_Alps_Hybrid:MX-1U-NoLED
- K6: value #5 -> 5; footprint MX_Alps_Hybrid:MX-1U -> MX_Alps_Hybrid:MX-1U-NoLED
- K60, K63: footprint MX_Alps_Hybrid:MX-1.25U -> MX_Alps_Hybrid:MX-1.25U-NoLED
- K62: footprint MX_Alps_Hybrid:MX-6.5U -> MX_Alps_Hybrid:MX-6.5U-NoLED
- K7: value #6 -> 6; footprint MX_Alps_Hybrid:MX-1U -> MX_Alps_Hybrid:MX-1U-NoLED
- K8: value #7 -> 7; footprint MX_Alps_Hybrid:MX-1U -> MX_Alps_Hybrid:MX-1U-NoLED
- K9: value #8 -> 8; footprint MX_Alps_Hybrid:MX-1U -> MX_Alps_Hybrid:MX-1U-NoLED

Commit message: PCB Footprint switched to MX only, layout changed
Parts:
- K1, K10, K11, K12, K13, K15, K17, K18, K19, K2, K20, K21, K22, K23, K24, K25, K26, K27, K28, K3, K30, K32, K33, K34, K35, K36, K37, K38, K39, K4, K40, K41, K42, K44, K46, K47, K48, K49, K5, K50, K51, K52, K53, K54, K55, K57, K58, K6, K65, K66, K67, K7, K8, K9: footprint MX_Alps_Hybrid:MX-1U-NoLED -> Mx_Only:MX-Solderable-1U
- K14: footprint MX_Alps_Hybrid:MX-2U-NoLED -> Mx_Only:MX-Solderable-2U
- K16, K29, K59, K61: footprint MX_Alps_Hybrid:MX-1.5U-NoLED -> Mx_Only:MX-Solderable-1.5U
- K31, K56: footprint MX_Alps_Hybrid:MX-1.75U-NoLED -> Mx_Only:MX-Solderable-1.75U
- K43, K45: footprint MX_Alps_Hybrid:MX-2.25U-NoLED -> Mx_Only:MX-Solderable-2.25U
- K60, K63: footprint MX_Alps_Hybrid:MX-1.25U-NoLED -> Mx_Only:MX-Solderable-1.25U
- K62: footprint MX_Alps_Hybrid:MX-6.5U-NoLED -> Mx_Only:MX-Solderable-6.25U
- K64: footprint MX_Alps_Hybrid:MX-1U-NoLED -> Mx_Only:MX-Solderable-1.25U
